Commit message: add grount truth position using p3d for gazebo

File: description/urdf/imu.xacro (robot description, xacro)
@@ -5,5 +5,5 @@
         <parent link="chassis" />
         <child link="imu_link"/>
-        <origin xyz="0 0 0.175" rpy="0 0 0"/>
+        <origin xyz="0.1 0 0.175" rpy="0 0 0"/>
     </joint>
     <link name="imu_link">
@@ -30,7 +30,7 @@
         <sensor name="imu_sensor" type="imu">
           <always_on>true</always_on>
-          <update_rate>100</update_rate>
+          <update_rate>30</update_rate>
           <visualize>true</visualize>
-          <topic>__default_topic__</topic>
+          <topic>imu</topic>
           <plugin filename="libgazebo_ros_imu_sensor.so" name="imu_plugin">
             <topicName>imu</topicName>

File: description/urdf/robot.urdf.xacro (robot description, xacro)
@@ -10,4 +10,7 @@
   <xacro:include filename="$(find slam_bot)/description/urdf/diffbot.materials.xacro" />
   <xacro:include filename="$(find slam_bot)/description/urdf/imu.xacro" />
+  <!-- <xacro:if value="$(arg sim_mode)"> -->
+    <xacro:include filename="$(find slam_bot)/description/urdf/gazebo_ground_truth.xacro" />
+  <!-- </xacro:if> -->
   <xacro:if value="$(arg use_ros2_control)">
     <xacro:include filename="$(find slam_bot)/description/ros2_control/ros2_control.xacro" />
