Commit message: fix depth camera orientation and add worlds

File: description/urdf/depth_camera.xacro (robot description, xacro)
@@ -4,10 +4,9 @@
         <parent link="chassis" />
         <child link="front_cam_link"/>
-        <origin xyz="-0.1 0 ${chassis_height/2}" rpy="${pi/2} -${pi/2} -${pi/2}"/>
+        <origin xyz="${chassis_length+0.1} 0 ${chassis_height+0.2}" rpy="0 0 0"/>
     </joint>
     <link name="front_cam_link">
         <visual>
             <box size="0.1 0.03 0.02"/>
-            <material name="red"/>
         </visual>
         <collision>

Commit message: fix depth camera orientation with camera_link_optical

File: description/urdf/depth_camera.xacro (robot description, xacro)
@@ -1,4 +1,5 @@
 <?xml version="1.0"?>
 <robot xmlns:xacro="http://www.ros.org/wiki/xacro">
+<<<<<<< HEAD
   <xacro name="pi" value="3.14159265359" />
   <joint name="front_cam_joint" type="fixed">
@@ -15,7 +16,31 @@
     </collision>
     <!-- <xacro:inertial_cylinder mass="0.1" length="0.04" radius="0.05">
+=======
+    <joint name="front_cam_joint" type="fixed">
+        <parent link="chassis" />
+        <child link="front_cam_link" />
+        <origin xyz="${chassis_length+0.1} 0 ${chassis_height+0.2}" rpy="0 0 0" />
+    </joint>
+    <joint name="camera_optical_joint" type="fixed">
+        <!-- these values have to be these values otherwise the gazebo camera
+            image won't be aligned properly with the frame it is supposedly
+            originating from -->
+        <origin xyz="0 0 0" rpy="${-pi/2} 0 ${-pi/2}" />
+        <parent link="front_cam_link" />
+        <child link="camera_link_optical" />
+    </joint>
+    <link name="front_cam_link">
+        <visual>
+            <box size="0.1 0.03 0.02" />
+        </visual>
+        <collision>
+            <box size="0.1 0.03 0.02" />
+        </collision>
+        <!-- <xacro:inertial_cylinder mass="0.1" length="0.04" radius="0.05">
+>>>>>>> e5fbb46 (fix depth camera orientation with camera_link_optical)
             <origin xyz="0 0 0" rpy="0 0 0"/>
         </xacro:inertial_cylinder> -->
   </link>
+<<<<<<< HEAD
   <joint name="camera_optical_joint" type="fixed">
     <!-- these values have to be these values otherwise the gazebo camera
@@ -57,3 +82,36 @@
     </sensor>
   </gazebo>
+=======
+    <link name="camera_link_optical">
+    </link>
+    <gazebo reference="front_cam_link">
+        <sensor name="front_camera" type="depth">
+            <always_on>1</always_on>
+            <visualize>1</visualize>
+            <update_rate>30</update_rate>
+            <camera>
+                <horizontal_fov>1.019272</horizontal_fov>
+                <image>
+                    <width>640</width>
+                    <height>480</height>
+                    <format>B8G8R8</format>
+                </image>
+                <clip>
+                    <near>0.2</near>
+                    <far>8</far>
+                </clip>
+            </camera>
+            <plugin name="camera_front" filename="libgazebo_ros_camera.so">
+                <ros>
+                    <namespace>diffbot</namespace>
+                </ros>
+                <frame_name>camera_link_optical</frame_name>
+                <camera_name>front</camera_name>
+                <hack_baseline>0.07</hack_baseline>
+                <min_depth>0.05</min_depth>
+                <max_depth>20.0</max_depth>
+            </plugin>
+        </sensor>
+    </gazebo>
+>>>>>>> e5fbb46 (fix depth camera orientation with camera_link_optical)
 </robot>

Commit message: add depth to laser scan converter

File: description/urdf/depth_camera.xacro (robot description, xacro)
@@ -1,20 +1,4 @@
 <?xml version="1.0"?>
 <robot xmlns:xacro="http://www.ros.org/wiki/xacro">
-<<<<<<< HEAD
-  <xacro name="pi" value="3.14159265359" />
-  <joint name="front_cam_joint" type="fixed">
-    <parent link="chassis" />
-    <child link="front_cam_link" />
-    <origin xyz="0.15 0 0.2" rpy="0 0 0" />
-  </joint>
-  <link name="front_cam_link">
-    <visual>
-      <box size="0.1 0.03 0.02" />
-    </visual>
-    <collision>
-      <box size="0.1 0.03 0.02" />
-    </collision>
-    <!-- <xacro:inertial_cylinder mass="0.1" length="0.04" radius="0.05">
-=======
     <joint name="front_cam_joint" type="fixed">
         <parent link="chassis" />
@@ -38,49 +22,7 @@
         </collision>
         <!-- <xacro:inertial_cylinder mass="0.1" length="0.04" radius="0.05">
->>>>>>> e5fbb46 (fix depth camera orientation with camera_link_optical)
             <origin xyz="0 0 0" rpy="0 0 0"/>
         </xacro:inertial_cylinder> -->
   </link>
-<<<<<<< HEAD
-  <joint name="camera_optical_joint" type="fixed">
-    <!-- these values have to be these values otherwise the gazebo camera
-          image won't be aligned properly with the frame it is supposedly
-          originating from -->
-    <origin xyz="0 0 0" rpy="${-pi/2} 0 ${-pi/2}" />
-    <parent link="front_cam_link" />
-    <child link="camera_link_optical" />
-  </joint>
-  <link name="camera_link_optical">
-  </link>
-  <gazebo reference="front_cam_link">
-    <sensor name="front_camera" type="depth">
-      <always_on>1</always_on>
-      <visualize>1</visualize>
-      <update_rate>30</update_rate>
-      <camera>
-        <horizontal_fov>1.019272</horizontal_fov>
-        <image>
-          <width>640</width>
-          <height>480</height>
-          <format>B8G8R8</format>
-        </image>
-        <clip>
-          <near>0.2</near>
-          <far>8</far>
-        </clip>
-      </camera>
-      <plugin name="camera_front" filename="libgazebo_ros_camera.so">
-        <ros>
-          <namespace>omni_bot</namespace>
-        </ros>
-        <frame_name>camera_link_optical</frame_name>
-        <camera_name>front</camera_name>
-        <hack_baseline>0.07</hack_baseline>
-        <min_depth>0.05</min_depth>
-        <max_depth>20.0</max_depth>
-      </plugin>
-    </sensor>
-  </gazebo>
-=======
     <link name="camera_link_optical">
     </link>
@@ -112,6 +54,29 @@
                 <max_depth>20.0</max_depth>
             </plugin>
+            <!-- <plugin name="camera_front" filename="libgazebo_ros_openni_kinect.so">
+              <baseline>0.2</baseline>
+              <alwaysOn>true</alwaysOn>
+              <updateRate>0.0</updateRate>
+              <cameraName>camera_ir</cameraName>
+              <imageTopicName>/camera/color/image_raw</imageTopicName>
+              <cameraInfoTopicName>/camera/color/camera_info</cameraInfoTopicName>
+              <depthImageTopicName>/camera/depth/image_raw</depthImageTopicName>
+              <depthImageCameraInfoTopicName>/camera/depth/camera_info</depthImageCameraInfoTopicName>
+              <pointCloudTopicName>/camera/depth/points</pointCloudTopicName>
+              <frameName>camera_link_optical</frameName>
+              <pointCloudCutoff>0.5</pointCloudCutoff>
+              <pointCloudCutoffMax>3.0</pointCloudCutoffMax>
+              <distortionK1>0</distortionK1>
+              <distortionK2>0</distortionK2>
+              <distortionK3>0</distortionK3>
+              <distortionT1>0</distortionT1>
+              <distortionT2>0</distortionT2>
+              <CxPrime>0</CxPrime>
+              <Cx>0</Cx>
+              <Cy>0</Cy>
+              <focalLength>0</focalLength>
+              <hackBaseline>0</hackBaseline>
+            </plugin> -->
         </sensor>
     </gazebo>
->>>>>>> e5fbb46 (fix depth camera orientation with camera_link_optical)
 </robot>
