Commit message: update omnibot size

File: description/omni_urdf/base/base.urdf.xacro (robot description, xacro)
@@ -11,5 +11,5 @@
           <visual>
                 <geometry>
-                  <box size="0.6 0.6 0.02" />
+                  <box size="0.3 0.3 0.02" />
                 </geometry>
                 <material name="white"/>
@@ -17,5 +17,5 @@
           <collision>
                 <geometry>
-                  <box size="0.6 0.6 0.02" />
+                  <box size="0.3 0.3 0.02" />
                 </geometry>
           </collision>

File: description/omni_urdf/robot.urdf.xacro (robot description, xacro)
@@ -2,5 +2,5 @@
 <robot name="omnibot" xmlns:xacro="http://ros.org/wiki/xacro">
   <xacro:arg name="prefix" default="" />
-  <xacro:arg name="use_sim" default="false" />
+  <xacro:arg name="use_sim" default="true" />
   <xacro:arg name="robot_name" default="omnibot"/>
   <xacro:include filename="$(find slam_bot)/description/omni_urdf/common.xacro"/>
@@ -18,17 +18,17 @@
   <!-- Wheel0 -->
   <xacro:omni_wheel prefix="wheel0" parent="base_link">
-	  <origin xyz="0.35 0.35 0.05" rpy="0 ${pi/2} ${pi/4}"/>
+	  <origin xyz="0.15 0.15 0.05" rpy="0 ${pi/2} ${pi/4}"/>
   </xacro:omni_wheel>
   <!-- Wheel1 -->
   <xacro:omni_wheel prefix="wheel1" parent="base_link">
-	  <origin xyz="-0.35 0.35 0.05" rpy="0 ${pi/2} ${pi*3/4}"/>
+	  <origin xyz="-0.15 0.15 0.05" rpy="0 ${pi/2} ${pi*3/4}"/>
   </xacro:omni_wheel>
   <!-- Wheel3 -->
   <xacro:omni_wheel prefix="wheel2" parent="base_link">
-	  <origin xyz="-0.35 -0.35 0.05" rpy="0 ${pi/2} ${-pi*3/4}"/>
+	  <origin xyz="-0.15 -0.15 0.05" rpy="0 ${pi/2} ${-pi*3/4}"/>
   </xacro:omni_wheel>
   <!-- Wheel2 -->
   <xacro:omni_wheel prefix="wheel3" parent="base_link">
-	  <origin xyz="0.35 -0.35 0.05" rpy="0 ${pi/2} ${-pi/4}"/>
+	  <origin xyz="0.15 -0.15 0.05" rpy="0 ${pi/2} ${-pi/4}"/>
   </xacro:omni_wheel>
   <!-- Base -->
@@ -38,5 +38,5 @@
   <!--<xacro:wheel_gazebo_v0 prefix="left"/>-->
   <!--xacro:wheel_gazebo_control_v0 rate="25"/-->
-  <joint name="camera_joint" type="fixed">
+  <!-- <joint name="camera_joint" type="fixed">
     <parent link="base_link"/>
     <child  link="camera_link"/>
@@ -52,4 +52,6 @@
     </visual>
   </link>
+   -->
+  <xacro:include filename="$(find slam_bot)/description/omni_urdf/depth_camera.xacro"/>
   <xacro:omnibot_gazebo prefix=""/>
   <xacro:omnibot_ros2_control name="omnibot" use_sim="$(arg use_sim)"/>

File: description/omni_urdf/wheel/wheel_100mm_light.urdf.xacro (robot description, xacro)
@@ -42,5 +42,5 @@
       <material>Gazebo/Gray</material>
       <mu1>0.8</mu1>
-      <mu2>0.05</mu2>
+      <mu2>0.2</mu2>
       <fdir1>0 1.0 0</fdir1>
       <kp value="30000000.0" />
