Commit message: fix camera optical orientation on rviz

File: description/omni_urdf/depth_camera.xacro (robot description, xacro)
@@ -1,48 +1,59 @@
 <?xml version="1.0"?>
-<robot xmlns:xacro="http://www.ros.org/wiki/xacro" >
-    <joint name="front_cam_joint" type="fixed">
-        <parent link="base_frame_link" />
-        <child link="front_cam_link"/>
-        <origin xyz="0.15 0 0" rpy="0 0 0"/>
-    </joint>
-    <link name="front_cam_link">
-        <visual>
-            <box size="0.1 0.03 0.02"/>
-        </visual>
-        <collision>
-            <box size="0.1 0.03 0.02"/>
-        </collision>
-        <!-- <xacro:inertial_cylinder mass="0.1" length="0.04" radius="0.05">
+<robot xmlns:xacro="http://www.ros.org/wiki/xacro">
+  <xacro name="pi" value="3.14159265359" />
+  <joint name="front_cam_joint" type="fixed">
+    <parent link="base_frame_link" />
+    <child link="front_cam_link" />
+    <origin xyz="0.15 0 0" rpy="0 0 0" />
+  </joint>
+  <link name="front_cam_link">
+    <visual>
+      <box size="0.1 0.03 0.02" />
+    </visual>
+    <collision>
+      <box size="0.1 0.03 0.02" />
+    </collision>
+    <!-- <xacro:inertial_cylinder mass="0.1" length="0.04" radius="0.05">
             <origin xyz="0 0 0" rpy="0 0 0"/>
         </xacro:inertial_cylinder> -->
-    </link>
-    <gazebo reference="front_cam_link">
-        <sensor name="front_camera" type="depth">
-          <always_on>1</always_on>
-          <visualize>1</visualize>
-          <update_rate>30</update_rate>
-          <camera>
-            <horizontal_fov>1.019272</horizontal_fov>
-            <image>
-              <width>640</width>
-              <height>480</height>
-              <format>B8G8R8</format>
-            </image>
-            <clip>
-              <near>0.2</near>
-              <far>8</far>
-            </clip>
-          </camera>
-          <plugin name="camera_front" filename="libgazebo_ros_camera.so">
-            <ros>
-              <namespace>omni_bot</namespace>
-            </ros>
-            <frame_name>front_cam_link</frame_name>
-            <camera_name>front</camera_name>
-            <hack_baseline>0.07</hack_baseline>
-            <min_depth>0.05</min_depth>
-            <max_depth>20.0</max_depth>
-          </plugin>
-        </sensor>
-      </gazebo>
+  </link>
+  <joint name="camera_optical_joint" type="fixed">
+    <!-- these values have to be these values otherwise the gazebo camera
+          image won't be aligned properly with the frame it is supposedly
+          originating from -->
+    <origin xyz="0 0 0" rpy="${-pi/2} 0 ${-pi/2}" />
+    <parent link="front_cam_link" />
+    <child link="camera_link_optical" />
+  </joint>
+  <link name="camera_link_optical">
+  </link>
+  <gazebo reference="front_cam_link">
+    <sensor name="front_camera" type="depth">
+      <always_on>1</always_on>
+      <visualize>1</visualize>
+      <update_rate>30</update_rate>
+      <camera>
+        <horizontal_fov>1.019272</horizontal_fov>
+        <image>
+          <width>640</width>
+          <height>480</height>
+          <format>B8G8R8</format>
+        </image>
+        <clip>
+          <near>0.2</near>
+          <far>8</far>
+        </clip>
+      </camera>
+      <plugin name="camera_front" filename="libgazebo_ros_camera.so">
+        <ros>
+          <namespace>omni_bot</namespace>
+        </ros>
+        <frame_name>camera_link_optical</frame_name>
+        <camera_name>front</camera_name>
+        <hack_baseline>0.07</hack_baseline>
+        <min_depth>0.05</min_depth>
+        <max_depth>20.0</max_depth>
+      </plugin>
+    </sensor>
+  </gazebo>
 </robot>

Commit message: add IMU link to omni bot

File: description/omni_urdf/depth_camera.xacro (robot description, xacro)
@@ -5,5 +5,5 @@
     <parent link="base_frame_link" />
     <child link="front_cam_link" />
-    <origin xyz="0.15 0 0" rpy="0 0 0" />
+    <origin xyz="0.15 0 0.2" rpy="0 0 0" />
   </joint>
   <link name="front_cam_link">

File: description/omni_urdf/robot.urdf.xacro (robot description, xacro)
@@ -54,4 +54,5 @@
    -->
   <xacro:include filename="$(find slam_bot)/description/omni_urdf/depth_camera.xacro"/>
+  <xacro:include filename="$(find slam_bot)/description/omni_urdf/imu.xacro"/>
   <xacro:omnibot_gazebo prefix=""/>
   <xacro:omnibot_ros2_control name="omnibot" use_sim="$(arg use_sim)"/>

File: description/urdf/depth_camera.xacro (robot description, xacro)
@@ -1,48 +1,59 @@
 <?xml version="1.0"?>
-<robot xmlns:xacro="http://www.ros.org/wiki/xacro" >
-    <joint name="front_cam_joint" type="fixed">
-        <parent link="chassis" />
-        <child link="front_cam_link"/>
-        <origin xyz="${chassis_length+0.1} 0 ${chassis_height+0.2}" rpy="0 0 0"/>
-    </joint>
-    <link name="front_cam_link">
-        <visual>
-            <box size="0.1 0.03 0.02"/>
-        </visual>
-        <collision>
-            <box size="0.1 0.03 0.02"/>
-        </collision>
-        <!-- <xacro:inertial_cylinder mass="0.1" length="0.04" radius="0.05">
+<robot xmlns:xacro="http://www.ros.org/wiki/xacro">
+  <xacro name="pi" value="3.14159265359" />
+  <joint name="front_cam_joint" type="fixed">
+    <parent link="chassis" />
+    <child link="front_cam_link" />
+    <origin xyz="0.15 0 0.2" rpy="0 0 0" />
+  </joint>
+  <link name="front_cam_link">
+    <visual>
+      <box size="0.1 0.03 0.02" />
+    </visual>
+    <collision>
+      <box size="0.1 0.03 0.02" />
+    </collision>
+    <!-- <xacro:inertial_cylinder mass="0.1" length="0.04" radius="0.05">
             <origin xyz="0 0 0" rpy="0 0 0"/>
         </xacro:inertial_cylinder> -->
-    </link>
-    <gazebo reference="front_cam_link">
-        <sensor name="front_camera" type="depth">
-          <always_on>1</always_on>
-          <visualize>1</visualize>
-          <update_rate>30</update_rate>
-          <camera>
-            <horizontal_fov>1.019272</horizontal_fov>
-            <image>
-              <width>640</width>
-              <height>480</height>
-              <format>B8G8R8</format>
-            </image>
-            <clip>
-              <near>0.2</near>
-              <far>8</far>
-            </clip>
-          </camera>
-          <plugin name="camera_front" filename="libgazebo_ros_camera.so">
-            <ros>
-              <namespace>slam_bot</namespace>
-            </ros>
-            <frame_name>front_cam_link</frame_name>
-            <camera_name>front</camera_name>
-            <hack_baseline>0.07</hack_baseline>
-            <min_depth>0.05</min_depth>
-            <max_depth>20.0</max_depth>
-          </plugin>
-        </sensor>
-      </gazebo>
+  </link>
+  <joint name="camera_optical_joint" type="fixed">
+    <!-- these values have to be these values otherwise the gazebo camera
+          image won't be aligned properly with the frame it is supposedly
+          originating from -->
+    <origin xyz="0 0 0" rpy="${-pi/2} 0 ${-pi/2}" />
+    <parent link="front_cam_link" />
+    <child link="camera_link_optical" />
+  </joint>
+  <link name="camera_link_optical">
+  </link>
+  <gazebo reference="front_cam_link">
+    <sensor name="front_camera" type="depth">
+      <always_on>1</always_on>
+      <visualize>1</visualize>
+      <update_rate>30</update_rate>
+      <camera>
+        <horizontal_fov>1.019272</horizontal_fov>
+        <image>
+          <width>640</width>
+          <height>480</height>
+          <format>B8G8R8</format>
+        </image>
+        <clip>
+          <near>0.2</near>
+          <far>8</far>
+        </clip>
+      </camera>
+      <plugin name="camera_front" filename="libgazebo_ros_camera.so">
+        <ros>
+          <namespace>omni_bot</namespace>
+        </ros>
+        <frame_name>camera_link_optical</frame_name>
+        <camera_name>front</camera_name>
+        <hack_baseline>0.07</hack_baseline>
+        <min_depth>0.05</min_depth>
+        <max_depth>20.0</max_depth>
+      </plugin>
+    </sensor>
+  </gazebo>
 </robot>

Commit message: update omnibot camera orientation and wheel friction

File: description/omni_urdf/depth_camera.xacro (robot description, xacro)
@@ -5,5 +5,5 @@
     <parent link="base_frame_link" />
     <child link="front_cam_link" />
-    <origin xyz="0.15 0 0.2" rpy="0 0 0" />
+    <origin xyz="-0.15 0 0.2" rpy="0 0 ${pi}" />
   </joint>
   <link name="front_cam_link">

File: description/omni_urdf/wheel/wheel_100mm_light.urdf.xacro (robot description, xacro)
@@ -42,5 +42,5 @@
       <material>Gazebo/Gray</material>
       <mu1>0.8</mu1>
-      <mu2>0.2</mu2>
+      <mu2>0.05</mu2>
       <fdir1>0 1.0 0</fdir1>
       <kp value="30000000.0" />
