Commit message: add velocity remapper

File: description/omni_urdf/lidar.xacro (robot description, xacro)
@@ -26,5 +26,5 @@
             <pose>0 0 0 0 0 0</pose>
             <visualize>true</visualize>
-            <update_rate>10</update_rate>
+            <update_rate>1000</update_rate>
             <ray>
                 <scan>

File: description/omni_urdf/robot.urdf.xacro (robot description, xacro)
@@ -53,7 +53,8 @@
   </link>
    -->
+  <xacro:include filename="$(find slam_bot)/description/omni_urdf/inertial_macros.xacro"/>
   <xacro:include filename="$(find slam_bot)/description/omni_urdf/depth_camera.xacro"/>
   <xacro:include filename="$(find slam_bot)/description/omni_urdf/imu.xacro"/>
-  <!-- <xacro:include filename="$(find slam_bot)/description/omni_urdf/lidar.xacro"/> -->
+  <xacro:include filename="$(find slam_bot)/description/omni_urdf/lidar.xacro"/>
   <xacro:omnibot_gazebo prefix=""/>
   <xacro:omnibot_ros2_control name="omnibot" use_sim="$(arg use_sim)"/>

File: description/urdf/depth_camera.xacro (robot description, xacro)
@@ -2,5 +2,5 @@
 <robot xmlns:xacro="http://www.ros.org/wiki/xacro">
     <joint name="front_cam_joint" type="fixed">
-        <parent link="chassis" />
+        <parent link="base_frame_link" />
         <child link="front_cam_link" />
         <origin xyz="${chassis_length+0.1} 0 ${chassis_height+0.2}" rpy="0 0 0" />
@@ -36,5 +36,5 @@
                 <image>
                     <width>640</width>
-                    <height>480</height>
+                    <height>400</height>
                     <format>B8G8R8</format>
                 </image>
@@ -46,5 +46,5 @@
             <plugin name="camera_front" filename="libgazebo_ros_camera.so">
                 <ros>
-                    <namespace>diffbot</namespace>
+                    <namespace>omni_bot</namespace>
                 </ros>
                 <frame_name>camera_link_optical</frame_name>

File: description/urdf/imu.xacro (robot description, xacro)
@@ -3,5 +3,5 @@
 <robot xmlns:xacro="http://www.ros.org/wiki/xacro" >
     <joint name="imu_joint" type="fixed">
-        <parent link="chassis" />
+        <parent link="base_frame_link" />
         <child link="imu_link"/>
         <origin xyz="0.1 0 0.175" rpy="0 0 0"/>

File: description/urdf/lidar.xacro (robot description, xacro)
@@ -2,5 +2,5 @@
 <robot xmlns:xacro="http://www.ros.org/wiki/xacro" >
     <joint name="laser_joint" type="fixed">
-        <parent link="chassis" />
+        <parent link="base_frame_link" />
         <child link="laser_frame"/>
         <origin xyz="0.1 0 0.175" rpy="0 0 0"/>

File: description/urdf/robot.urdf.xacro (robot description, xacro)
@@ -11,4 +11,5 @@
   <xacro:include filename="$(find slam_bot)/description/urdf/imu.xacro" />
   <xacro:include filename="$(find slam_bot)/description/urdf/depth_camera.xacro" />
+  <xacro:include filename="$(find slam_bot)/description/urdf/lidar.xacro" />
   <!-- <xacro:if value="$(arg sim_mode)"> -->
     <xacro:include filename="$(find slam_bot)/description/urdf/gazebo_ground_truth.xacro" />

File: description/urdf/robot_core.xacro (robot description, xacro)
@@ -33,17 +33,17 @@
     </material> -->
     <!-- BASE LINK -->
-    <link name="base_link">
+    <link name="base_frame_link">
     </link>
     <!-- BASE_FOOTPRINT LINK -->
     <joint name="base_footprint_joint" type="fixed">
-        <parent link="base_link"/>
-        <child link="base_footprint"/>
+        <parent link="base_frame_link"/>
+        <child link="base_link"/>
         <origin xyz="0 0 0" rpy="0 0 0"/>
     </joint>
-    <link name="base_footprint">
+    <link name="base_link">
     </link>
     <!-- CHASSIS LINK -->
     <joint name="chassis_joint" type="fixed">
-        <parent link="base_link"/>
+        <parent link="base_frame_link"/>
         <child link="chassis"/>
         <origin xyz="${-wheel_offset_x} 0 ${-wheel_offset_z}"/>
