Commit message: fix simulation launch and add IMU

File: description/ros2_control/ros2_control.xacro (robot description, xacro)
@@ -35,10 +35,16 @@
       </xacro:if>
       <joint name="${prefix}left_wheel_joint">
-        <command_interface name="velocity" />
+        <command_interface name="velocity">
+          <param name="min">-10</param>
+          <param name="max">10</param>
+        </command_interface>
         <state_interface name="position" />
         <state_interface name="velocity" />
       </joint>
       <joint name="${prefix}right_wheel_joint">
-        <command_interface name="velocity" />
+        <command_interface name="velocity">
+          <param name="min">-10</param>
+          <param name="max">10</param>
+        </command_interface>
         <state_interface name="position" />
         <state_interface name="velocity" />
@@ -57,9 +63,15 @@
       </sensor> -->
     </ros2_control>
-    <xacro:if value="${use_mock_hardware}">
+    <gazebo>
+      <plugin name="gazebo_ros2_control" filename="libgazebo_ros2_control.so">
+        <parameters>$(find slam_bot)/config/diffbot_controllers.yaml</parameters>
+        <parameters>$(find slam_bot)/config/gaz_ros2_ctl_use_sim.yaml</parameters>
+      </plugin>
+    </gazebo>
+    <!-- <xacro:if value="${use_mock_hardware}">
       <plugin filename="ign_ros2_control-system" name="ign_ros2_control::IgnitionROS2ControlPlugin">
         <parameters>$(find slam_bot)/config/diffbot_controllers.yaml</parameters>
       </plugin>
-    </xacro:if>
+    </xacro:if> -->
   </xacro:macro>
 </robot>

File: description/urdf/robot.urdf.xacro (robot description, xacro)
@@ -6,6 +6,8 @@
   <xacro:arg name="use_ros2_control" default="true"/>
   <xacro:include filename="$(find slam_bot)/description/urdf/robot_core.xacro" />
+  <xacro:include filename="$(find slam_bot)/description/urdf/inertial_macros.xacro" />
   <!-- Import Rviz colors -->
   <xacro:include filename="$(find slam_bot)/description/urdf/diffbot.materials.xacro" />
+  <xacro:include filename="$(find slam_bot)/description/urdf/imu.xacro" />
   <xacro:if value="$(arg use_ros2_control)">
     <xacro:include filename="$(find slam_bot)/description/ros2_control/ros2_control.xacro" />

File: description/urdf/robot_core.xacro (robot description, xacro)
@@ -1,163 +1,151 @@
 <?xml version="1.0"?>
-<robot xmlns:xacro="http://www.ros.org/wiki/xacro">
-  <xacro:macro name="diffbot" params="prefix">
-    <!-- Constants for robot dimensions -->
-    <xacro:property name="PI" value="3.1415926535897931" />
-    <xacro:property name="base_mass" value="0.3" /> <!-- arbitrary value for base mass -->
-    <xacro:property name="base_width" value="0.3" />
-    <xacro:property name="base_length" value="0.24" />
-    <xacro:property name="base_height" value="0.12" />
-    <xacro:property name="wheel_mass" value="0.3" /> <!-- arbitrary value for wheel mass -->
-    <xacro:property name="wheel_len" value="0.020" />
-    <xacro:property name="wheel_radius" value="0.03" />
-    <xacro:property name="caster_wheel_mass" value="0.1" /> <!-- arbitrary value for caster wheel mass -->
-    <xacro:property name="caster_wheel_radius" value="0.015" />
-    <xacro:property name="z_offset" value="0" /> <!-- Space btw top of beam and the each joint -->
-    <!-- Base Link -->
-    <link name="${prefix}base_link">
-      <collision>
-        <origin xyz="0 0 0" rpy="0 0 0" />
-        <geometry>
-          <box size="${base_width} ${base_length} ${base_height}" />
-        </geometry>
-      </collision>
-      <visual>
-        <origin xyz="0 0 ${base_height/2}" rpy="0 0 0" />
-        <geometry>
-          <box size="${base_width} ${base_length} ${base_height}" />
-        </geometry>
-        <material name="orange" />
-      </visual>
-      <inertial>
-        <origin xyz="0 0 0" rpy="0 0 0" />
-        <mass value="${base_mass}" />
-        <inertia
-          ixx="${base_mass / 12.0 * (base_length*base_length + base_height*base_height)}" ixy="0.0"
-          ixz="0.0"
-          iyy="${base_mass / 12.0 * (base_height*base_height + base_width*base_width)}" iyz="0.0"
-          izz="${base_mass / 12.0 * (base_width*base_width + base_length*base_length)}" />
-      </inertial>
+<robot xmlns:xacro="http://www.ros.org/wiki/xacro" >
+    <xacro:macro name="diffbot" params="prefix"/>
+    <xacro:include filename="inertial_macros.xacro"/>
+    <xacro:property name="chassis_length" value="0.335"/>
+    <xacro:property name="chassis_width" value="0.265"/>
+    <xacro:property name="chassis_height" value="0.138"/>
+    <xacro:property name="chassis_mass" value="1.0"/>
+    <xacro:property name="wheel_radius" value="0.033"/>
+    <xacro:property name="wheel_thickness" value="0.026"/>
+    <xacro:property name="wheel_mass" value="0.05"/>
+    <xacro:property name="wheel_offset_x" value="0.226"/>
+    <xacro:property name="wheel_offset_y" value="0.1485"/>
+    <xacro:property name="wheel_offset_z" value="0.01"/>
+    <xacro:property name="caster_wheel_radius" value="0.01"/>
+    <xacro:property name="caster_wheel_mass" value="0.01"/>
+    <xacro:property name="caster_wheel_offset_x" value="0.075"/>
+    <xacro:property name="caster_wheel_offset_z" value="${wheel_offset_z - wheel_radius + caster_wheel_radius}"/>
+    <!-- <material name="white">
+        <color rgba="1 1 1 1" />
+    </material>
+    <material name="orange">
+        <color rgba="1 0.3 0.1 1"/>
+    </material>
+    <material name="blue">
+        <color rgba="0.2 0.2 1 1"/>
+    </material>
+    <material name="black">
+        <color rgba="0 0 0 1"/>
+    </material>
+    <material name="red">
+        <color rgba="1 0 0 1"/>
+    </material> -->
+    <!-- BASE LINK -->
+    <link name="base_link">
     </link>
-    <joint name="${prefix}left_wheel_joint" type="continuous">
-      <parent link="${prefix}base_link" />
-      <child link="${prefix}left_wheel" />
-      <origin xyz="-${base_length/2-wheel_radius} -${base_width/2} ${z_offset}" rpy="0 0 0" />
-      <axis xyz="0 1 0" />
-      <dynamics damping="0.2" />
+    <!-- BASE_FOOTPRINT LINK -->
+    <joint name="base_footprint_joint" type="fixed">
+        <parent link="base_link"/>
+        <child link="base_footprint"/>
+        <origin xyz="0 0 0" rpy="0 0 0"/>
     </joint>
-    <!-- left wheel Link -->
-    <link name="${prefix}left_wheel">
-      <collision>
-        <origin xyz="0 0 0" rpy="${PI/2} 0 0" />
-        <geometry>
-          <cylinder length="${wheel_len}" radius="${wheel_radius}" />
-        </geometry>
-      </collision>
-      <visual>
-        <origin xyz="0 0 0" rpy="${PI/2} 0 0" />
-        <geometry>
-          <cylinder length="${wheel_len}" radius="${wheel_radius}" />
-        </geometry>
-        <material name="black" />
-      </visual>
-      <inertial>
-        <origin xyz="0 0 0" rpy="${PI/2} 0 0" />
-        <mass value="${wheel_mass}" />
-        <inertia
-          ixx="${wheel_mass / 12.0 * (3*wheel_radius + wheel_len*wheel_len)}" ixy="0.0" ixz="0.0"
-          iyy="${wheel_mass / 12.0 * wheel_radius*wheel_radius}" iyz="0.0"
-          izz="${wheel_mass / 12.0 * wheel_radius*wheel_radius}" />
-      </inertial>
+    <link name="base_footprint">
     </link>
-    <joint name="${prefix}right_wheel_joint" type="continuous">
-      <parent link="${prefix}base_link" />
-      <child link="${prefix}right_wheel" />
-      <origin xyz="-${base_length/2-wheel_radius} ${base_width/2} ${z_offset}" rpy="0 0 0" />
-      <axis xyz="0 1 0" />
-      <dynamics damping="0.2" />
+    <!-- CHASSIS LINK -->
+    <joint name="chassis_joint" type="fixed">
+        <parent link="base_link"/>
+        <child link="chassis"/>
+        <origin xyz="${-wheel_offset_x} 0 ${-wheel_offset_z}"/>
     </joint>
-    <!-- right wheel Link -->
-    <link name="${prefix}right_wheel">
-      <collision>
-        <origin xyz="0 0 0" rpy="${PI/2} 0 0" />
-        <geometry>
-          <cylinder length="${wheel_len}" radius="${wheel_radius}" />
-        </geometry>
-      </collision>
-      <visual>
-        <origin xyz="0 0 0" rpy="${PI/2} 0 0" />
-        <geometry>
-          <cylinder length="${wheel_len}" radius="${wheel_radius}" />
-        </geometry>
-        <material name="black" />
-      </visual>
-      <inertial>
-        <origin xyz="0 0 0" rpy="${PI/2} 0 0" />
-        <mass value="${wheel_mass}" />
-        <inertia
-          ixx="${wheel_mass / 12.0 * (3*wheel_radius + wheel_len*wheel_len)}" ixy="0.0" ixz="0.0"
-          iyy="${wheel_mass / 12.0 * wheel_radius*wheel_radius}" iyz="0.0"
-          izz="${wheel_mass / 12.0 * wheel_radius*wheel_radius}" />
-      </inertial>
+    <link name="chassis">
+        <visual>
+            <origin xyz="${chassis_length/2} 0 ${chassis_height/2}"/>
+            <geometry>
+                <box size="${chassis_length} ${chassis_width} ${chassis_height}"/>
+            </geometry>
+            <material name="orange"/>
+        </visual>
+        <collision>
+            <origin xyz="${chassis_length/2} 0 ${chassis_height/2}"/>
+            <geometry>
+                <box size="${chassis_length} ${chassis_width} ${chassis_height}"/>
+            </geometry>
+        </collision>
+        <xacro:inertial_box mass="0.5" x="${chassis_length}" y="${chassis_width}" z="${chassis_height}">
+            <origin xyz="${chassis_length/2} 0 ${chassis_height/2}" rpy="0 0 0"/>
+        </xacro:inertial_box>
     </link>
-    <joint name="${prefix}caster_frontal_wheel_joint" type="fixed">
-      <parent link="${prefix}base_link" />
-      <child link="${prefix}caster_frontal_wheel" />
-      <origin xyz="${base_width/2 - caster_wheel_radius} 0 ${z_offset}" rpy="0 0 0" />
+    <gazebo reference="chassis">
+        <material>Gazebo/Orange</material>
+    </gazebo>
+    <!-- LEFT WHEEL LINK -->
+    <joint name="left_wheel_joint" type="continuous">
+        <parent link="base_link"/>
+        <child link="left_wheel"/>
+        <origin xyz="0 ${wheel_offset_y} 0" rpy="-${pi/2} 0 0" />
+        <axis xyz="0 0 1"/>
     </joint>
-    <!-- caster frontal wheel Link -->
-    <link name="${prefix}caster_frontal_wheel">
-      <collision>
-        <origin xyz="0 0 0" rpy="0 0 0" />
-        <geometry>
-          <sphere radius="${caster_wheel_radius}" />
-        </geometry>
-      </collision>
-      <visual>
-        <origin xyz="0 0 0" rpy="0 0 0" />
-        <geometry>
-          <sphere radius="${caster_wheel_radius}" />
-        </geometry>
-        <material name="white" />
-      </visual>
-      <inertial>
-        <origin xyz="0 0 0" rpy="0 0 0" />
-        <mass value="${caster_wheel_mass}" />
-        <inertia
-          ixx="${caster_wheel_mass * 0.4 * (caster_wheel_radius * caster_wheel_radius)}" ixy="0.0"
-          ixz="0.0"
-          iyy="${caster_wheel_mass * 0.4 * (caster_wheel_radius * caster_wheel_radius)}" iyz="0.0"
-          izz="${caster_wheel_mass * 0.4 * (caster_wheel_radius * caster_wheel_radius)}" />
-      </inertial>
+    <link name="left_wheel">
+        <visual>
+            <geometry>
+                <cylinder radius="${wheel_radius}" length="${wheel_thickness}"/>
+            </geometry>
+            <material name="blue"/>
+        </visual>
+        <collision>
+            <geometry>
+                <sphere radius="${wheel_radius}"/>
+            </geometry>
+        </collision>
+        <xacro:inertial_cylinder mass="${wheel_mass}" length="${wheel_thickness}" radius="${wheel_radius}">
+            <origin xyz="0 0 0" rpy="0 0 0"/>
+        </xacro:inertial_cylinder>
     </link>
-    <!-- <joint name="${prefix}caster_rear_wheel_joint" type="fixed">
-      <parent link="${prefix}base_link"/>
-      <child link="${prefix}caster_rear_wheel"/>
-      <origin xyz="${-base_width/2 + caster_wheel_radius} 0 ${z_offset}" rpy="0 0 0"/>
-    </joint> -->
-    <!-- caster rear wheel Link -->
-    <!-- <link name="${prefix}caster_rear_wheel">
-      <collision>
-        <origin xyz="0 0 0" rpy="0 0 0"/>
-        <geometry>
-          <sphere radius="${caster_wheel_radius}"/>
-        </geometry>
-      </collision>
-      <visual>
-        <origin xyz="0 0 0" rpy="0 0 0"/>
-        <geometry>
-          <sphere radius="${caster_wheel_radius}"/>
-        </geometry>
-        <material name="white"/>
-      </visual>
-      <inertial>
-        <origin xyz="0 0 0" rpy="0 0 0"/>
-        <mass value="${caster_wheel_mass}"/>
-        <inertia
-          ixx="${caster_wheel_mass * 0.4 * (caster_wheel_radius * caster_wheel_radius)}" ixy="0.0" ixz="0.0"
-          iyy="${caster_wheel_mass * 0.4 * (caster_wheel_radius * caster_wheel_radius)}" iyz="0.0"
-          izz="${caster_wheel_mass * 0.4 * (caster_wheel_radius * caster_wheel_radius)}"/>
-        </inertial>
-      </link> -->
-  </xacro:macro>
+    <gazebo reference="left_wheel">
+        <material>Gazebo/Blue</material>
+    </gazebo>
+    <!-- RIGHT WHEEL LINK -->
+    <joint name="right_wheel_joint" type="continuous">
+        <parent link="base_link"/>
+        <child link="right_wheel"/>
+        <origin xyz="0 ${-wheel_offset_y} 0" rpy="${pi/2} 0 0" />
+        <axis xyz="0 0 -1"/>
+    </joint>
+    <link name="right_wheel">
+        <visual>
+            <geometry>
+                <cylinder radius="${wheel_radius}" length="${wheel_thickness}"/>
+            </geometry>
+            <material name="blue"/>
+        </visual>
+        <collision>
+            <geometry>
+                <sphere radius="${wheel_radius}"/>
+            </geometry>
+        </collision>
+        <xacro:inertial_cylinder mass="${wheel_mass}" length="${wheel_thickness}" radius="${wheel_radius}">
+            <origin xyz="0 0 0" rpy="0 0 0"/>
+        </xacro:inertial_cylinder>
+    </link>
+    <gazebo reference="right_wheel">
+        <material>Gazebo/Blue</material>
+    </gazebo>
+    <!-- CASTER WHEEL LINK -->
+    <joint name="caster_wheel_joint" type="fixed">
+        <parent link="chassis"/>
+        <child link="caster_wheel"/>
+        <origin xyz="${caster_wheel_offset_x} 0 ${caster_wheel_offset_z}"/>
+    </joint>
+    <link name="caster_wheel">
+        <visual>
+            <geometry>
+                <sphere radius="${caster_wheel_radius}"/>
+            </geometry>
+            <material name="white"/>
+        </visual>
+        <collision>
+            <geometry>
+                <sphere radius="${caster_wheel_radius}"/>
+            </geometry>
+        </collision>
+        <xacro:inertial_sphere mass="${caster_wheel_mass}" radius="${caster_wheel_radius}">
+            <origin xyz="0 0 0" rpy="0 0 0"/>
+        </xacro:inertial_sphere>
+    </link>
+    <gazebo reference="caster_wheel">
+        <material>Gazebo/White</material>
+        <mu1 value="0.001"/>
+        <mu2 value="0.001"/>
+    </gazebo>
 </robot>

Commit message: update readme

File: description/ros2_control/ros2_control.xacro (robot description, xacro)
@@ -34,5 +34,5 @@
         </hardware>
       </xacro:if>
-      <joint name="${prefix}left_wheel_joint">
+      <joint name="left_wheel_joint">
         <command_interface name="velocity">
           <param name="min">-10</param>
@@ -42,5 +42,5 @@
         <state_interface name="velocity" />
       </joint>
-      <joint name="${prefix}right_wheel_joint">
+      <joint name="right_wheel_joint">
         <command_interface name="velocity">
           <param name="min">-10</param>

File: description/urdf/robot.urdf.xacro (robot description, xacro)
@@ -11,5 +11,5 @@
   <xacro:include filename="$(find slam_bot)/description/urdf/imu.xacro" />
   <xacro:include filename="$(find slam_bot)/description/urdf/depth_camera.xacro" />
-  <xacro:include filename="$(find slam_bot)/description/urdf/lidar.xacro" />
+  <!-- <xacro:include filename="$(find slam_bot)/description/urdf/lidar.xacro" /> -->
   <!-- <xacro:if value="$(arg sim_mode)"> -->
     <xacro:include filename="$(find slam_bot)/description/urdf/gazebo_ground_truth.xacro" />
